File: espusb/esp8266sch.sch (KiCad schematic (older format))
At the start: 17 parts, among them CON1 SD_Card, P4 CONN_02X04, P5 CONN_01X03, U3 esp8266, U4 SERFLASH, X1 CRYSTAL_SMD

Commit message: missing link to antenna and ground
Parts:
- A1: symbol CONN_01X01 -> CONN_01X02
Connections:
- net GND: now also A1.2 (P2)
Changed lines of the file:
@@
 	1700 3500 2450 3500
 $Comp
-L CONN_01X01 A1
+L CONN_01X02 A1
 U 1 1 572B16C9
-P 1700 3300
-F 0 "A1" H 1700 3400 50  0000 C CNN
-F 1 "antenna" V 1800 3300 50  0000 C CNN
-F 2 "wifiantenna:wifi_antenna" H 1700 3300 60  0001 C CNN
-F 3 "" H 1700 3300 60  0000 C CNN
-	1    1700 3300
+P 1750 3200
+F 0 "A1" H 1750 3300 50  0000 C CNN
+F 1 "antenna" V 1850 3200 50  0000 C CNN
+F 2 "wifiantenna:wifi_antenna" H 1750 3200 60  0001 C CNN
+F 3 "" H 1750 3200 60  0000 C CNN
+	1    1750 3200
 	0    -1   -1   0
 $EndComp
@@
 Wire Wire Line
 	5200 2550 4500 2550
+Wire Wire Line
+	1700 3500 1700 3400
+$Comp
+L GND #PWR?
+U 1 1 572C423A
+P 1800 3600
+F 0 "#PWR?" H 1800 3350 50  0001 C CNN
+F 1 "GND" H 1800 3450 50  0000 C CNN
+F 2 "" H 1800 3600 60  0000 C CNN
+F 3 "" H 1800 3600 60  0000 C CNN
+	1    1800 3600
+	1    0    0    -1
+$EndComp
+Wire Wire Line
+	1800 3600 1800 3400
 $EndSCHEMATC

Commit message: current version
Parts:
- added C10: 10uF, Capacitors_SMD:C_0805, symbol C
- added R1: 10K, Resistors_SMD:R_0603, symbol R
Connections:
- net +3V3: now also C10.2, R1.1
- net GND: now also C10.1; no longer CON1.3 (VSS), CON1.9 (DAT2)
- net GPIO4: now also CON1.2 (CMD); no longer CON1.1 (CD/DAT3)
- net MTCK: now also CON1.3 (VSS); no longer CON1.2 (CMD)
- net MTDI: now also R1.2
Other:
- moved on the sheet: CON1
Changed lines of the file:
@@
 L SD_Card CON1
 U 1 1 572B8B7B
-P 2000 6550
-F 0 "CON1" H 1350 7100 50  0000 C CNN
-F 1 "SD_Card" H 2600 6000 50  0000 C CNN
-F 2 "microsd:MICROSD" H 2200 6900 50  0000 C CNN
-F 3 "" H 2000 6550 60  0000 C CNN
-	1    2000 6550
+P 2100 6550
+AR Path="/572B8B7B" Ref="CON1"  Part="1"
+AR Path="/572B01F2/572B8B7B" Ref="CON1"  Part="1"
+F 0 "CON1" H 1450 7100 50  0000 C CNN
+F 1 "SD_Card" H 2700 6000 50  0000 C CNN
+F 2 "microsd:MICROSD" H 2300 6900 50  0000 C CNN
+F 3 "" H 2100 6550 60  0000 C CNN
+	1    2100 6550
 	-1   0    0    1
 $EndComp
-Wire Wire Line
-	2900 6550 3500 6550
-Wire Wire Line
-	3500 6550 3500 6300
 $Comp
 L +3.3V #PWR028
 U 1 1 572B8EEB
-P 3500 6300
-F 0 "#PWR028" H 3500 6150 50  0001 C CNN
-F 1 "+3.3V" H 3500 6440 50  0000 C CNN
-F 2 "" H 3500 6300 60  0000 C CNN
-F 3 "" H 3500 6300 60  0000 C CNN
-	1    3500 6300
-	1    0    0    -1
-$EndComp
-Wire Wire Line
-	2900 6650 3500 6650
-Wire Wire Line
-	3500 6650 3500 6700
+P 4000 6500
+F 0 "#PWR028" H 4000 6350 50  0001 C CNN
+F 1 "+3.3V" H 4000 6640 50  0000 C CNN
+F 2 "" H 4000 6500 60  0000 C CNN
+F 3 "" H 4000 6500 60  0000 C CNN
+	1    4000 6500
+	1    0    0    -1
+$EndComp
 $Comp
 L GND #PWR029
-U 1 1 572B8FD9
-P 3500 6700
-F 0 "#PWR029" H 3500 6450 50  0001 C CNN
-F 1 "GND" H 3500 6550 50  0000 C CNN
-F 2 "" H 3500 6700 60  0000 C CNN
-F 3 "" H 3500 6700 60  0000 C CNN
-	1    3500 6700
-	1    0    0    -1
-$EndComp
-$Comp
-L GND #PWR030
 U 1 1 572B9031
-P 3350 6400
-F 0 "#PWR030" H 3350 6150 50  0001 C CNN
-F 1 "GND" H 3250 6300 50  0000 C CNN
-F 2 "" H 3350 6400 60  0000 C CNN
-F 3 "" H 3350 6400 60  0000 C CNN
-	1    3350 6400
-	1    0    0    -1
-$EndComp
-Wire Wire Line
-	3350 6400 3350 6350
-Wire Wire Line
-	3350 6350 2900 6350
+P 3800 6300
+F 0 "#PWR029" H 3800 6050 50  0001 C CNN
+F 1 "GND" H 3700 6200 50  0000 C CNN
+F 2 "" H 3800 6300 60  0000 C CNN
+F 3 "" H 3800 6300 60  0000 C CNN
+	1    3800 6300
+	1    0    0    -1
+$EndComp
 Text GLabel 3700 4800 0    60   Input ~ 0
 MTDI
-Text GLabel 3050 6250 2    60   Input ~ 0
+Text GLabel 3350 6200 2    60   Input ~ 0
 MTDI
-Wire Wire Line
-	3050 6250 2900 6250
 Text GLabel 3700 4650 0    60   Input ~ 0
 MTMS
-Text GLabel 3650 6400 2    60   Input ~ 0
+Text GLabel 3350 6400 2    60   Input ~ 0
 MTMS
-Wire Wire Line
-	2950 6400 3650 6400
-Wire Wire Line
-	2950 6400 2950 6450
-Wire Wire Line
-	2950 6450 2900 6450
 Wire Wire Line
 	5950 5350 6600 5350
@@
 Wire Wire Line
 	3750 4950 3700 4950
-Wire Wire Line
-	2900 6750 3300 6750
-Wire Wire Line
-	3300 6750 3300 6950
-Wire Wire Line
-	3300 6950 3700 6950
-Text GLabel 3700 6950 2    60   Input ~ 0
+Text GLabel 3350 6600 2    60   Input ~ 0
 MTCK
 $Comp
-L +3.3V #PWR031
+L +3.3V #PWR030
 U 1 1 572BE61C
 P 5250 5100
-F 0 "#PWR031" H 5250 4950 50  0001 C CNN
+F 0 "#PWR030" H 5250 4950 50  0001 C CNN
 F 1 "+3.3V" H 5250 5240 50  0000 C CNN
 F 2 "" H 5250 5100 60  0000 C CNN
@@
 Text GLabel 6350 4600 2    60   Input ~ 0
 GPIO4
-Text GLabel 3250 7100 2    60   Input ~ 0
+Text GLabel 3350 6800 2    60   Input ~ 0
 GPIO4
-Wire Wire Line
-	3250 7100 3150 7100
-Wire Wire Line
-	3150 7100 3150 6850
-Wire Wire Line
-	3150 6850 2900 6850
 $Comp
 L esp8266 U3
@@
 Wire Wire Line
 	2100 2650 2250 2650
-$Comp
-L GND #PWR032
-U 1 1 572C93DA
-P 2900 7050
-F 0 "#PWR032" H 2900 6800 50  0001 C CNN
-F 1 "GND" H 2900 6900 50  0000 C CNN
-F 2 "" H 2900 7050 60  0000 C CNN
-F 3 "" H 2900 7050 60  0000 C CNN
-	1    2900 7050
-	1    0    0    -1
-$EndComp
-Wire Wire Line
-	2900 7050 2900 6950
 Wire Wire Line
 	5200 2550 4500 2550
@@
 	1700 3500 1700 3400
 $Comp
-L GND #PWR033
+L GND #PWR031
 U 1 1 572C423A
 P 1800 3600
-F 0 "#PWR033" H 1800 3350 50  0001 C CNN
+F 0 "#PWR031" H 1800 3350 50  0001 C CNN
 F 1 "GND" H 1800 3450 50  0000 C CNN
 F 2 "" H 1800 3600 60  0000 C CNN
@@
 Wire Wire Line
 	1800 3600 1800 3400
+Wire Wire Line
+	3350 6800 3300 6800
+Wire Wire Line
+	3300 6800 3300 6750
+Wire Wire Line
+	3300 6750 3000 6750
+Wire Wire Line
+	3350 6600 3300 6600
+Wire Wire Line
+	3300 6600 3300 6650
+Wire Wire Line
+	3300 6650 3000 6650
+Wire Wire Line
+	4000 6500 3300 6500
+Wire Wire Line
+	3300 6500 3300 6550
+Wire Wire Line
+	3300 6550 3000 6550
+Wire Wire Line
+	3350 6400 3250 6400
+Wire Wire Line
+	3250 6400 3250 6450
+Wire Wire Line
+	3250 6450 3000 6450
+Wire Wire Line
+	3800 6300 3200 6300
+Wire Wire Line
+	3200 6300 3200 6350
+Wire Wire Line
+	3200 6350 3000 6350
+Wire Wire Line
+	3350 6200 3150 6200
+Wire Wire Line
+	3150 6200 3150 6250
+Wire Wire Line
+	3150 6250 3000 6250
+$Comp
+L R R1
+U 1 1 575A873A
+P 3250 6000
+F 0 "R1" V 3330 6000 50  0000 C CNN
+F 1 "10K" V 3250 6000 50  0000 C CNN
+F 2 "Resistors_SMD:R_0603" V 3180 6000 30  0001 C CNN
+F 3 "" H 3250 6000 30  0000 C CNN
+	1    3250 6000
+	1    0    0    -1
+$EndComp
+Wire Wire Line
+	3250 6150 3250 6200
+Connection ~ 3250 6200
+$Comp
+L +3.3V #PWR032
+U 1 1 575A8879
+P 3250 5800
+F 0 "#PWR032" H 3250 5650 50  0001 C CNN
+F 1 "+3.3V" H 3250 5940 50  0000 C CNN
+F 2 "" H 3250 5800 60  0000 C CNN
+F 3 "" H 3250 5800 60  0000 C CNN
+	1    3250 5800
+	1    0    0    -1
+$EndComp
+Wire Wire Line
+	3250 5800 3250 5850
+$Comp
+L C C10
+U 1 1 575CE3FB
+P 4250 6400
+F 0 "C10" H 4275 6500 50  0000 L CNN
+F 1 "10uF" H 4275 6300 50  0000 L CNN
+F 2 "Capacitors_SMD:C_0805" H 4288 6250 30  0001 C CNN
+F 3 "" H 4250 6400 60  0000 C CNN
+	1    4250 6400
+	1    0    0    -1
+$EndComp
+Wire Wire Line
+	4250 6250 3800 6250
+Wire Wire Line
+	3800 6250 3800 6300
+Wire Wire Line
+	4250 6550 3950 6550
+Wire Wire Line
+	3950 6550 3950 6500
+Connection ~ 3950 6500
 $EndSCHEMATC
