File: BabySeq/BabySeq.kicad_pcb (KiCad board)
At the start: 2 copper layers, 100.2 x 100.2 mm, 62 parts, among them P1 SPEAKERCON, P2 PWRCON, SW1 SWITCH_INV, SW2 SWITCH_INV, SW3 SWITCH_INV, U1 LM555N, U2 LM555N, U3 LM555N, U4 4017

Commit message: misc
Other:
- board size 100.2 x 100.2 mm -> 100 x 100 mm
Changed lines of the file:
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@@
     (links 100)
     (no_connects 0)
-    (area 152.218619 13.821 283.429 127.000001)
+    (area 152.218619 12.621 283.429 127.000001)
     (thickness 1.6)
-    (drawings 23)
+    (drawings 26)
     (tracks 291)
     (zones 0)
@@
   (page A4)
   (layers
-    (0 F.Cu signal)
-    (31 B.Cu signal)
+    (0 F.Cu signal hide)
+    (31 B.Cu signal hide)
     (32 B.Adhes user)
     (33 F.Adhes user)
@@
     (pad "" thru_hole circle (at -4 0 90) (size 1.524 1.524) (drill 1.1) (layers *.Cu *.Mask F.SilkS))
   )
+  (gr_arc (start 212 69) (end 212 19) (angle 90) (layer Edge.Cuts) (width 0.1))
+  (gr_arc (start 212 69) (end 162 69) (angle 90) (layer Edge.Cuts) (width 0.1))
+  (gr_arc (start 212 69) (end 212 119) (angle 90) (layer Edge.Cuts) (width 0.1))
+  (gr_arc (start 212 69) (end 262 69) (angle 90) (layer Edge.Cuts) (width 0.1))
   (gr_text 10uF (at 204.4 96) (layer F.SilkS)
     (effects (font (size 1 1) (thickness 0.15)))
@@
     (effects (font (size 1.5 1.5) (thickness 0.3)))
   )
-  (gr_circle (center 212 69) (end 257 91) (layer Edge.Cuts) (width 0.1))
   (gr_circle (center 212 73.5) (end 168 82.5) (layer Dwgs.User) (width 0.1))
   (gr_text "Whiteford Research Limited\nPunkSeq10 - r2" (at 240 75.8) (layer B.SilkS)
