File: stm_pcbs/a9ref/a9ref/a9ref.kicad_pcb (KiCad board)
At the start: 2 copper layers, 50.2 x 44.5 mm, 25 parts, among them J400 CONN_5, J401 CONN_5, Q401 2n3904, U1 LTZ1000A, U2 LT1013

Commit message: current
Other:
- board text added: "a9 r3"
Changed lines of the file:
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@@
   (general
     (thickness 1.6)
-    (drawings 11)
+    (drawings 12)
     (tracks 219)
     (zones 0)
@@
     (pad 1 np_thru_hole circle (at 0 0) (size 4.3 4.3) (drill 4.3) (layers *.Cu *.Mask))
   )
+  (gr_text "a9 r3" (at 139.065 167.64) (layer F.SilkS)
+    (effects (font (size 1.5 1.5) (thickness 0.3)))
+  )
   (gr_line (start 164.465 170.18) (end 119.38 170.18) (angle 90) (layer Edge.Cuts) (width 0.15))
