File: ddc112brd/ddc112brd.kicad_pcb (KiCad board)
At the start: 2 copper layers, 91.4 x 71.1 mm, 22 parts, among them P1 BNC, P2 BNC, P3 CONN_20X2, U1 AD8675, U2 ddc112, U3 A9_REFERENCE, U4 TXCO

Commit message: DDC112 board, multislope and various other updates it seems
Parts:
- P1, P2: footprint sma:SMA -> stmshieldfull:SMA
Other:
- board text added: "MAKE POWER TRACES THICKER"
