File: stm_pcbs/stm_integrated/ADC.sch (KiCad schematic (older format))
At the start: 10 parts, among them P5 BNC, U16 LT1019ACS8, U17 LTC1859

Commit message: working on Kicad of 3rd Dec
Parts:
- C77, C78, C79, C80, C81, C82: symbol C -> device:C
- P5: symbol BNC -> device:BNC
- R10: symbol R -> device:R
- U16: symbol LT1019ACS8 -> LTC1859:LT1019ACS8
- U17: symbol LTC1859 -> LTC1859:LTC1859
Connections:
- net labels added: ADC_BUSY, ADC_CONVST, ADC_RD, SCLK, SDIN, SDO
- wire segments 49 -> 63
Changed lines of the file:
@@
-EESchema Schematic File Version 2
-LIBS:power
-LIBS:device
-LIBS:transistors
-LIBS:conn
-LIBS:linear
-LIBS:regul
-LIBS:74xx
-LIBS:cmos4000
-LIBS:adc-dac
-LIBS:memory
-LIBS:xilinx
-LIBS:special
-LIBS:microcontrollers
-LIBS:dsp
-LIBS:microchip
-LIBS:analog_switches
-LIBS:motorola
-LIBS:texas
-LIBS:intel
-LIBS:audio
-LIBS:interface
-LIBS:digital-audio
-LIBS:philips
-LIBS:display
-LIBS:cypress
-LIBS:siliconi
-LIBS:opto
-LIBS:atmel
-LIBS:contrib
-LIBS:valves
-LIBS:ad5791
+EESchema Schematic File Version 4
 LIBS:stmshieldfull-cache
-LIBS:powerbrd-cache
-LIBS:LTC1859-cache
-EELAYER 25 0
+EELAYER 26 0
 EELAYER END
 $Descr A4 11693 8268
@@
 $EndDescr
 $Comp
-L LTC1859 U17
+L LTC1859:LTC1859 U17
 U 1 1 5A233DCE
 P 5250 3600
@@
 $EndComp
 $Comp
-L C C78
+L device:C C78
 U 1 1 5A233DDC
 P 3950 3300
@@
 $EndComp
 $Comp
-L AGND #PWR060
+L power:AGND #PWR060
 U 1 1 5A233E0D
 P 4550 4450
@@
 $EndComp
 $Comp
-L AGND #PWR061
+L power:AGND #PWR061
 U 1 1 5A233E13
 P 6550 4100
@@
 $EndComp
 $Comp
-L DGND #PWR062
+L power:DGND #PWR062
 U 1 1 5A233E19
-P 6400 3450
-F 0 "#PWR062" H 6400 3450 40  0001 C CNN
-F 1 "DGND" H 6400 3380 40  0000 C CNN
-F 2 "" H 6400 3450 60  0000 C CNN
-F 3 "" H 6400 3450 60  0000 C CNN
-	1    6400 3450
-	1    0    0    -1
-$EndComp
-$Comp
-L C C80
+P 6750 3350
+F 0 "#PWR062" H 6750 3350 40  0001 C CNN
+F 1 "DGND" H 6750 3280 40  0000 C CNN
+F 2 "" H 6750 3350 60  0000 C CNN
+F 3 "" H 6750 3350 60  0000 C CNN
+	1    6750 3350
+	1    0    0    -1
+$EndComp
+$Comp
+L device:C C80
 U 1 1 5A233E1F
 P 6150 4500
@@
 $EndComp
 $Comp
-L AGND #PWR063
+L power:AGND #PWR063
 U 1 1 5A233E26
 P 6150 4800
@@
 $EndComp
 $Comp
-L AGND #PWR064
+L power:AGND #PWR064
 U 1 1 5A233E2C
 P 3950 3600
@@
 $EndComp
 $Comp
-L AGND #PWR065
+L power:AGND #PWR065
 U 1 1 5A233E39
 P 4450 2750
@@
 $EndComp
 $Comp
-L +5V #PWR066
+L power:+5V #PWR066
 U 1 1 5A233E3F
 P 7150 3750
@@
 $EndComp
 $Comp
-L C C81
+L device:C C81
 U 1 1 5A233E45
 P 6850 4050
@@
 $EndComp
 $Comp
-L C C82
+L device:C C82
 U 1 1 5A233E4C
 P 7050 4050
@@
 $EndComp
 $Comp
-L DGND #PWR067
+L power:DGND #PWR067
 U 1 1 5A233E53
 P 6950 4600
@@
 $EndComp
 $Comp
-L LT1019ACS8 U16
+L LTC1859:LT1019ACS8 U16
 U 1 1 5A233E59
 P 4100 5450
@@
 $EndComp
 $Comp
-L C C77
+L device:C C77
 U 1 1 5A233E60
 P 3250 5600
@@
 $EndComp
 $Comp
-L C C79
+L device:C C79
 U 1 1 5A233E67
 P 5250 5800
@@
 $EndComp
 $Comp
-L AGND #PWR068
+L power:AGND #PWR068
 U 1 1 5A233E6E
 P 5100 6000
@@
 $EndComp
 $Comp
-L AGND #PWR069
+L power:AGND #PWR069
 U 1 1 5A233E74
 P 3550 5800
@@
 $EndComp
 $Comp
-L +5V #PWR070
+L power:+5V #PWR070
 U 1 1 5A233E7A
 P 3250 5300
@@
 $EndComp
 $Comp
-L BNC P5
+L device:BNC P5
 U 1 1 5A233EB5
 P 3500 3050
@@
 $EndComp
 $Comp
-L AGND #PWR071
+L power:AGND #PWR071
 U 1 1 5A233F90
 P 7850 4450
@@
 $EndComp
 $Comp
-L DGND #PWR072
+L power:DGND #PWR072
 U 1 1 5A233F96
 P 8400 4450
@@
 $EndComp
 $Comp
-L AGND #PWR073
+L power:AGND #PWR073
 U 1 1 5A233F9E
 P 3250 5800
@@
 $EndComp
 $Comp
-L R R10
+L device:R R10
 U 1 1 5A233FA7
 P 8150 4300
@@
 	6150 3950 6150 4050
 Wire Wire Line
-	5900 4050 6550 4050
+	5900 4050 6150 4050
 Wire Wire Line
 	6550 4050 6550 4100
 Connection ~ 6150 4050
 Wire Wire Line
-	5900 3350 6400 3350
-Wire Wire Line
-	6400 3350 6400 3450
-Wire Wire Line
 	6150 4650 6150 4800
 Wire Wire Line
@@
 	6150 4150 5900 4150
 Wire Wire Line
-	3650 3050 4550 3050
+	3650 3050 3950 3050
 Wire Wire Line
 	3950 3050 3950 3150
@@
 	5900 3650 6100 3650
 Wire Wire Line
-	6100 3650 6100 3850
+	6100 3650 6100 3750
 Wire Wire Line
 	6100 3850 5900 3850
 Wire Wire Line
-	5900 3750 7150 3750
+	5900 3750 6100 3750
 Connection ~ 6100 3750
 Wire Wire Line
 	6950 4600 6950 4250
 Wire Wire Line
-	6850 4250 7050 4250
+	6850 4250 6950 4250
 Connection ~ 6950 4250
 Wire Wire Line
-	4650 5500 5900 5500
+	4650 5500 5250 5500
 Wire Wire Line
 	5900 5500 5900 4250
@@
 	3550 5600 3550 5800
 Wire Wire Line
-	3250 5300 3250 5450
+	3250 5300 3250 5400
 Connection ~ 3950 3050
 Wire Wire Line
@@
 Connection ~ 5250 5500
 Wire Wire Line
-	5900 2800 5900 3050
-Wire Wire Line
 	8400 4300 8400 4450
 Wire Wire Line
@@
 	8400 4300 8300 4300
 Wire Wire Line
-	3950 3450 3950 3600
+	3950 3450 3950 3500
 Wire Wire Line
 	3950 3500 3500 3500
@@
 Wire Wire Line
 	4450 2650 4450 2750
+Wire Wire Line
+	6150 4050 6550 4050
+Wire Wire Line
+	6100 3750 6100 3850
+Wire Wire Line
+	6100 3750 6850 3750
+Wire Wire Line
+	6950 4250 7050 4250
+Wire Wire Line
+	3950 3050 4550 3050
+Wire Wire Line
+	5250 5500 5900 5500
+Wire Wire Line
+	7050 3750 7150 3750
+Wire Wire Line
+	6850 3750 7050 3750
+Wire Wire Line
+	3250 5400 3250 5450
+Wire Wire Line
+	3950 3500 3950 3600
+Text GLabel 6050 2950 2    60   Input ~ 0
+ADC_CONVST
+Text GLabel 6050 3050 2    60   Input ~ 0
+ADC_RD
+Text GLabel 6050 3550 2    60   Input ~ 0
+ADC_BUSY
+Text GLabel 6050 3150 2    60   Input ~ 0
+SCLK
+Text GLabel 6050 3250 2    60   Input ~ 0
+SDIN
+Text GLabel 6050 3450 2    60   Input ~ 0
+SDO
+Wire Wire Line
+	5900 3350 6750 3350
+Wire Wire Line
+	6050 2950 5900 2950
+Wire Wire Line
+	5900 3050 6050 3050
+Wire Wire Line
+	6050 3150 5900 3150
+Wire Wire Line
+	5900 3250 6050 3250
+Wire Wire Line
+	6050 3450 5900 3450
+Wire Wire Line
+	5900 3550 6050 3550
 $EndSCHEMATC

Commit message: fixing more borkage
Connections:
- wire segments 63 -> 56
Changed lines of the file:
@@
 L power:AGND #PWR068
 U 1 1 5A233E6E
-P 5100 6000
-F 0 "#PWR068" H 5100 6000 40  0001 C CNN
-F 1 "AGND" H 5100 5930 50  0000 C CNN
-F 2 "" H 5100 6000 60  0000 C CNN
-F 3 "" H 5100 6000 60  0000 C CNN
-	1    5100 6000
+P 5250 6050
+F 0 "#PWR068" H 5250 6050 40  0001 C CNN
+F 1 "AGND" H 5250 5980 50  0000 C CNN
+F 2 "" H 5250 6050 60  0000 C CNN
+F 3 "" H 5250 6050 60  0000 C CNN
+	1    5250 6050
 	1    0    0    -1
 $EndComp
@@
 Connection ~ 6150 4050
 Wire Wire Line
-	6150 4650 6150 4800
-Wire Wire Line
-	6150 4150 6150 4350
-Wire Wire Line
 	6150 4150 5900 4150
-Wire Wire Line
-	3650 3050 3950 3050
-Wire Wire Line
-	3950 3050 3950 3150
 Wire Wire Line
 	4550 4250 4550 4450
@@
 Connection ~ 6950 4250
 Wire Wire Line
-	4650 5500 5250 5500
-Wire Wire Line
 	5900 5500 5900 4250
 Wire Wire Line
 	3600 5400 3250 5400
 Wire Wire Line
-	5100 6000 5250 6000
+	5250 6050 5250 6000
 Wire Wire Line
 	3600 5600 3550 5600
@@
 Wire Wire Line
 	3250 5300 3250 5400
-Connection ~ 3950 3050
-Wire Wire Line
-	5250 5500 5250 5650
-Connection ~ 5250 5500
 Wire Wire Line
 	8400 4300 8400 4450
 Wire Wire Line
-	7850 4300 8000 4300
+	7850 4300 7900 4300
 Wire Wire Line
 	7850 4300 7850 4450
 Wire Wire Line
-	7050 3750 7050 3900
-Connection ~ 7050 3750
-Wire Wire Line
-	6850 3750 6850 3900
+	6850 3750 6850 3850
 Connection ~ 6850 3750
-Wire Wire Line
-	5250 6000 5250 5950
 Connection ~ 3250 5400
-Wire Wire Line
-	3250 5750 3250 5800
-Wire Wire Line
-	6850 4200 6850 4250
-Wire Wire Line
-	7050 4250 7050 4200
-Wire Wire Line
-	8400 4300 8300 4300
-Wire Wire Line
-	3950 3450 3950 3500
 Wire Wire Line
 	3950 3500 3500 3500
@@
 Wire Wire Line
 	6950 4250 7050 4250
-Wire Wire Line
-	3950 3050 4550 3050
-Wire Wire Line
-	5250 5500 5900 5500
-Wire Wire Line
-	7050 3750 7150 3750
-Wire Wire Line
-	6850 3750 7050 3750
-Wire Wire Line
-	3250 5400 3250 5450
 Wire Wire Line
 	3950 3500 3950 3600
@@
 Wire Wire Line
 	5900 3550 6050 3550
+Wire Wire Line
+	6850 3750 7050 3750
+Wire Wire Line
+	7050 3850 7050 3750
+Connection ~ 7050 3750
+Wire Wire Line
+	7050 3750 7150 3750
+Wire Wire Line
+	4650 5500 5250 5500
+Wire Wire Line
+	5250 5600 5250 5500
+Connection ~ 5250 5500
+Wire Wire Line
+	5250 5500 5900 5500
+Wire Wire Line
+	3650 3050 3950 3050
+Wire Wire Line
+	3950 3100 3950 3050
+Connection ~ 3950 3050
+Wire Wire Line
+	3950 3050 4550 3050
+Wire Wire Line
+	6150 4300 6150 4150
+Wire Wire Line
+	6150 4800 6150 4700
 $EndSCHEMATC
