File: stm_pcbs/stm_integrated/DAC1.sch (KiCad schematic (older format))
At the start: 21 parts, among them P100 BNC, U100 AD5791, U101 AD8676, U102 AD8675

Commit message: Mostly Chua's stuff
Parts:
- C17, C19, C21, C23, C24, C27, C28, C31, C32: symbol device:C -> Device:C
- C18, C20, C22, C25, C26, C29, C30: symbol device:CP1 -> Device:CP
- P100: symbol device:BNC -> Connector:Conn_Coaxial
- R2: symbol device:R -> Device:R
Connections:
- net AGND renamed GNDA
- net DGND renamed GNDD
Changed lines of the file:
@@
 EESchema Schematic File Version 4
-LIBS:stmshieldfull-cache
-EELAYER 26 0
+EELAYER 30 0
 EELAYER END
 $Descr A4 11693 8268
@@
 $EndComp
 $Comp
-L device:BNC P100
+L Connector:Conn_Coaxial P100
 U 1 1 5A25DBDA
 P 7850 3550
@@
 -14V
 $Comp
-L power:AGND #PWR013
+L power:GNDA #PWR013
 U 1 1 5A25DBE7
 P 7850 3900
 F 0 "#PWR013" H 7850 3900 40  0001 C CNN
-F 1 "AGND" H 7850 3830 50  0000 C CNN
+F 1 "GNDA" H 7850 3830 50  0000 C CNN
 F 2 "" H 7850 3900 60  0000 C CNN
 F 3 "" H 7850 3900 60  0000 C CNN
@@
 -14V
 $Comp
-L power:AGND #PWR014
+L power:GNDA #PWR014
 U 1 1 5A25DBF0
 P 4850 5000
 F 0 "#PWR014" H 4850 5000 40  0001 C CNN
-F 1 "AGND" H 4850 4930 50  0000 C CNN
+F 1 "GNDA" H 4850 4850 50  0000 C CNN
 F 2 "" H 4850 5000 60  0000 C CNN
 F 3 "" H 4850 5000 60  0000 C CNN
@@
 $EndComp
 $Comp
-L power:DGND #PWR015
+L power:GNDD #PWR015
 U 1 1 5A25DBF6
 P 4600 5000
 F 0 "#PWR015" H 4600 5000 40  0001 C CNN
-F 1 "DGND" H 4600 4930 40  0000 C CNN
+F 1 "GNDD" H 4600 4850 40  0000 C CNN
 F 2 "" H 4600 5000 60  0000 C CNN
 F 3 "" H 4600 5000 60  0000 C CNN
@@
 $EndComp
 $Comp
-L device:C C19
+L Device:C C19
 U 1 1 5A25DBFC
 P 5850 2300
@@
 $EndComp
 $Comp
-L power:AGND #PWR016
+L power:GNDA #PWR016
 U 1 1 5A25DC03
 P 6300 2450
 F 0 "#PWR016" H 6300 2450 40  0001 C CNN
-F 1 "AGND" H 6300 2380 50  0000 C CNN
+F 1 "GNDA" H 6300 2300 50  0000 C CNN
 F 2 "" H 6300 2450 60  0000 C CNN
 F 3 "" H 6300 2450 60  0000 C CNN
@@
 $EndComp
 $Comp
-L device:C C21
+L Device:C C21
 U 1 1 5A25DC09
 P 6000 4650
@@
 $EndComp
 $Comp
-L power:AGND #PWR017
+L power:GNDA #PWR017
 U 1 1 5A25DC10
 P 6400 4850
 F 0 "#PWR017" H 6400 4850 40  0001 C CNN
-F 1 "AGND" H 6400 4780 50  0000 C CNN
+F 1 "GNDA" H 6400 4700 50  0000 C CNN
 F 2 "" H 6400 4850 60  0000 C CNN
 F 3 "" H 6400 4850 60  0000 C CNN
@@
 $EndComp
 $Comp
-L device:C C17
+L Device:C C17
 U 1 1 5A25DC24
 P 3850 2000
@@
 $EndComp
 $Comp
-L power:DGND #PWR018
+L power:GNDD #PWR018
 U 1 1 5A25DC2B
 P 3600 1800
 F 0 "#PWR018" H 3600 1800 40  0001 C CNN
-F 1 "DGND" H 3600 1730 40  0000 C CNN
+F 1 "GNDD" H 3600 1650 40  0000 C CNN
 F 2 "" H 3600 1800 60  0000 C CNN
 F 3 "" H 3600 1800 60  0000 C CNN
@@
 $EndComp
 $Comp
-L device:C C24
+L Device:C C24
 U 1 1 5A25DC31
 P 7350 5700
@@
 $EndComp
 $Comp
-L device:C C31
+L Device:C C31
 U 1 1 5A25DC38
 P 8750 5550
@@
 $EndComp
 $Comp
-L device:C C32
+L Device:C C32
 U 1 1 5A25DC3F
 P 8750 6100
@@
 $EndComp
 $Comp
-L power:AGND #PWR019
+L power:GNDA #PWR019
 U 1 1 5A25DC46
 P 9000 5800
 F 0 "#PWR019" H 9000 5800 40  0001 C CNN
-F 1 "AGND" H 9000 5730 50  0000 C CNN
+F 1 "GNDA" H 9000 5730 50  0000 C CNN
 F 2 "" H 9000 5800 60  0000 C CNN
 F 3 "" H 9000 5800 60  0000 C CNN
@@
 $EndComp
 $Comp
-L power:AGND #PWR020
+L power:GNDA #PWR020
 U 1 1 5A25DC4C
 P 9000 6350
 F 0 "#PWR020" H 9000 6350 40  0001 C CNN
-F 1 "AGND" H 9000 6280 50  0000 C CNN
+F 1 "GNDA" H 9000 6280 50  0000 C CNN
 F 2 "" H 9000 6350 60  0000 C CNN
 F 3 "" H 9000 6350 60  0000 C CNN
@@
 $EndComp
 $Comp
-L device:C C23
+L Device:C C23
 U 1 1 5A25DC52
 P 7100 5700
@@
 $EndComp
 $Comp
-L device:CP1 C29
+L Device:CP C29
 U 1 1 5A25DC59
 P 8500 5550
@@
 $EndComp
 $Comp
-L device:CP1 C30
+L Device:CP C30
 U 1 1 5A25DC60
 P 8500 6100
@@
 $EndComp
 $Comp
-L device:CP1 C22
+L Device:CP C22
 U 1 1 5A25DC67
 P 6000 5000
@@
 $EndComp
 $Comp
-L device:CP1 C20
+L Device:CP C20
 U 1 1 5A25DC6E
 P 5850 2550
@@
 $EndComp
 $Comp
-L device:CP1 C18
+L Device:CP C18
 U 1 1 5A25DC75
 P 4100 2000
@@
 RESET1
 $Comp
-L device:CP1 C25
+L Device:CP C25
 U 1 1 5A25DC83
 P 7400 3200
@@
 $EndComp
 $Comp
-L device:CP1 C26
+L Device:CP C26
 U 1 1 5A25DC8A
 P 7400 3950
@@
 $EndComp
 $Comp
-L device:C C27
+L Device:C C27
 U 1 1 5A25DC91
 P 7600 3200
@@
 $EndComp
 $Comp
-L device:C C28
+L Device:C C28
 U 1 1 5A25DC98
 P 7600 3950
@@
 $EndComp
 $Comp
-L power:AGND #PWR021
+L power:GNDA #PWR021
 U 1 1 5A25DC9F
 P 7300 3400
 F 0 "#PWR021" H 7300 3400 40  0001 C CNN
-F 1 "AGND" H 7300 3330 50  0000 C CNN
+F 1 "GNDA" H 7300 3330 50  0000 C CNN
 F 2 "" H 7300 3400 60  0000 C CNN
 F 3 "" H 7300 3400 60  0000 C CNN
@@
 $EndComp
 $Comp
-L power:AGND #PWR022
+L power:GNDA #PWR022
 U 1 1 5A25DCA5
 P 7400 4250
 F 0 "#PWR022" H 7400 4250 40  0001 C CNN
-F 1 "AGND" H 7400 4180 50  0000 C CNN
+F 1 "GNDA" H 7400 4180 50  0000 C CNN
 F 2 "" H 7400 4250 60  0000 C CNN
 F 3 "" H 7400 4250 60  0000 C CNN
@@
 Connection ~ 6850 3900
 $Comp
-L device:R R2
+L Device:R R2
 U 1 1 5A25DD1F
 P 7150 4550
@@
 $EndComp
 $Comp
-L power:AGND #PWR023
+L power:GNDA #PWR023
 U 1 1 5A25DD26
 P 6900 4750
 F 0 "#PWR023" H 6900 4750 40  0001 C CNN
-F 1 "AGND" H 6900 4680 50  0000 C CNN
+F 1 "GNDA" H 6900 4680 50  0000 C CNN
 F 2 "" H 6900 4750 60  0000 C CNN
 F 3 "" H 6900 4750 60  0000 C CNN
@@
 $EndComp
 $Comp
-L power:DGND #PWR024
+L power:GNDD #PWR024
 U 1 1 5A25DD2C
 P 7400 4750
 F 0 "#PWR024" H 7400 4750 40  0001 C CNN
-F 1 "DGND" H 7400 4680 40  0000 C CNN
+F 1 "GNDD" H 7400 4680 40  0000 C CNN
 F 2 "" H 7400 4750 60  0000 C CNN
 F 3 "" H 7400 4750 60  0000 C CNN
@@
 Wire Wire Line
 	7400 4250 7400 4150
-Connection ~ 8750 6300
-Connection ~ 8750 5750
-Wire Wire Line
-	7150 3550 7700 3550
 Wire Wire Line
 	4650 2500 4800 2500
@@
 	8750 5750 8750 5800
 Wire Wire Line
-	3850 2200 4100 2200
-Wire Wire Line
 	7250 6050 7700 6050
 Wire Wire Line
-	6850 3000 7400 3000
-Wire Wire Line
-	6850 3750 7400 3750
-Wire Wire Line
-	7300 3400 7400 3400
-Wire Wire Line
 	7400 4550 7400 4750
 Wire Wire Line
@@
 Wire Wire Line
 	5800 4650 5800 4800
-Connection ~ 7400 3000
-Wire Wire Line
-	7400 3000 7600 3000
-Connection ~ 7400 3400
-Wire Wire Line
-	7400 3400 7600 3400
-Connection ~ 7400 3750
-Wire Wire Line
-	7400 3750 7600 3750
-Connection ~ 7400 4150
 Wire Wire Line
 	5600 2050 5600 2300
-Wire Wire Line
-	5650 2300 5600 2300
 Connection ~ 5600 2300
 Wire Wire Line
 	5600 2300 5600 2400
-Connection ~ 4100 2200
-Wire Wire Line
-	4100 2200 4450 2200
 $Comp
 L power:+5V #PWR080
@@
 	4200 2400 4400 2400
 Wire Wire Line
-	7750 5900 8500 5900
-Connection ~ 8500 5900
-Wire Wire Line
-	8500 5900 8750 5900
-Wire Wire Line
 	7700 6050 7750 6050
 Connection ~ 7750 6050
 Wire Wire Line
 	7750 6050 7800 6050
+Wire Wire Line
+	3850 2200 4100 2200
+Wire Wire Line
+	6850 3000 7400 3000
+Wire Wire Line
+	6850 3750 7400 3750
+Wire Wire Line
+	7300 3400 7400 3400
+Wire Wire Line
+	7750 5900 8500 5900
+Wire Wire Line
+	4100 1850 4100 1800
+Wire Wire Line
+	3850 1800 3850 1850
+Wire Wire Line
+	3850 2150 3850 2200
+Wire Wire Line
+	4100 2150 4100 2200
+Connection ~ 4100 2200
+Wire Wire Line
+	4100 2200 4450 2200
+Wire Wire Line
+	6000 2550 6050 2550
+Wire Wire Line
+	6050 2300 6000 2300
+Wire Wire Line
+	5600 2300 5700 2300
+Wire Wire Line
+	5650 2550 5700 2550
+Wire Wire Line
+	5850 4650 5800 4650
+Wire Wire Line
+	5800 5000 5850 5000
+Wire Wire Line
+	6150 5000 6200 5000
+Wire Wire Line
+	6200 4650 6150 4650
+Wire Wire Line
+	7400 4550 7300 4550
+Wire Wire Line
+	7000 4550 6900 4550
+Wire Wire Line
+	7150 3550 7650 3550
+Connection ~ 7650 3550
+Wire Wire Line
+	7650 3550 7700 3550
+Wire Wire Line
+	7600 4100 7600 4150
+Wire Wire Line
+	7400 4100 7400 4150
+Connection ~ 7400 4150
+Wire Wire Line
+	7400 3800 7400 3750
+Connection ~ 7400 3750
+Wire Wire Line
+	7400 3750 7600 3750
+Wire Wire Line
+	7600 3800 7600 3750
+Wire Wire Line
+	7600 3350 7600 3400
+Wire Wire Line
+	7400 3350 7400 3400
+Connection ~ 7400 3400
+Wire Wire Line
+	7400 3400 7600 3400
+Wire Wire Line
+	7400 3050 7400 3000
+Connection ~ 7400 3000
+Wire Wire Line
+	7400 3000 7600 3000
+Wire Wire Line
+	7600 3050 7600 3000
+Wire Wire Line
+	8750 5400 8750 5350
+Wire Wire Line
+	8500 5350 8500 5400
+Wire Wire Line
+	8500 5700 8500 5750
+Wire Wire Line
+	8750 5700 8750 5750
+Connection ~ 8750 5750
+Wire Wire Line
+	8750 6250 8750 6300
+Connection ~ 8750 6300
+Wire Wire Line
+	8500 6250 8500 6300
+Wire Wire Line
+	8500 5950 8500 5900
+Connection ~ 8500 5900
+Wire Wire Line
+	8500 5900 8750 5900
+Wire Wire Line
+	8750 5900 8750 5950
+Wire Wire Line
+	7350 5550 7350 5500
+Wire Wire Line
+	7100 5500 7100 5550
+Wire Wire Line
+	7100 5850 7100 5900
+Wire Wire Line
+	7350 5850 7350 5900
 $EndSCHEMATC
