File: stm_pcbs/stm_integrated/DAC3.sch (KiCad schematic (older format))
At the start: 21 parts, among them P3 BNC, U7 AD8676, U8 AD5791, U9 AD8675

Commit message: working on Kicad of 3rd Dec
Parts:
- C33, C35, C37, C39, C40, C43, C44, C47, C48: symbol C -> device:C
- C34, C36, C38, C41, C42, C45, C46: symbol CP2 -> device:CP1
- P3: symbol BNC -> device:BNC
- R3: symbol R -> device:R
- U7: symbol AD8676 -> ad5791:AD8676
- U8: symbol AD5791 -> ad5791:AD5791
- U9: symbol AD8675 -> ad5791:AD8675
Connections:
- wire segments 111 -> 126
Changed lines of the file:
@@
-EESchema Schematic File Version 2
-LIBS:power
-LIBS:device
-LIBS:transistors
-LIBS:conn
-LIBS:linear
-LIBS:regul
-LIBS:74xx
-LIBS:cmos4000
-LIBS:adc-dac
-LIBS:memory
-LIBS:xilinx
-LIBS:special
-LIBS:microcontrollers
-LIBS:dsp
-LIBS:microchip
-LIBS:analog_switches
-LIBS:motorola
-LIBS:texas
-LIBS:intel
-LIBS:audio
-LIBS:interface
-LIBS:digital-audio
-LIBS:philips
-LIBS:display
-LIBS:cypress
-LIBS:siliconi
-LIBS:opto
-LIBS:atmel
-LIBS:contrib
-LIBS:valves
-LIBS:ad5791
+EESchema Schematic File Version 4
 LIBS:stmshieldfull-cache
-LIBS:powerbrd-cache
-LIBS:LTC1859-cache
-EELAYER 25 0
+EELAYER 26 0
 EELAYER END
 $Descr A4 11693 8268
@@
 $EndDescr
 $Comp
-L AD5791 U8
+L ad5791:AD5791 U8
 U 1 1 5A25F8A7
 P 5150 3800
@@
 $EndComp
 $Comp
-L AD8675 U9
+L ad5791:AD8675 U9
 U 1 1 5A25F8AE
 P 6850 3450
@@
 $EndComp
 $Comp
-L AD8676 U7
+L ad5791:AD8676 U7
 U 1 1 5A25F8B5
 P 5050 1750
@@
 $EndComp
 $Comp
-L AD8676 U7
+L ad5791:AD8676 U7
 U 2 1 5A25F8BC
 P 5100 5500
@@
 $EndComp
 $Comp
-L AD8676 U7
+L ad5791:AD8676 U7
 U 3 1 5A25F8C3
 P 7800 5600
@@
 $EndComp
 $Comp
-L BNC P3
+L device:BNC P3
 U 1 1 5A25F8CA
 P 7950 3450
@@
 -14V
 $Comp
-L AGND #PWR025
+L power:AGND #PWR025
 U 1 1 5A25F8D7
 P 7950 3800
@@
 3.3V
 $Comp
-L AGND #PWR026
+L power:AGND #PWR026
 U 1 1 5A25F8E0
 P 4950 4900
@@
 $EndComp
 $Comp
-L DGND #PWR027
+L power:DGND #PWR027
 U 1 1 5A25F8E6
 P 4700 4900
@@
 $EndComp
 $Comp
-L C C35
+L device:C C35
 U 1 1 5A25F8EC
 P 5950 2200
@@
 $EndComp
 $Comp
-L AGND #PWR028
+L power:AGND #PWR028
 U 1 1 5A25F8F3
 P 6400 2350
@@
 $EndComp
 $Comp
-L C C37
+L device:C C37
 U 1 1 5A25F8F9
 P 6100 4600
@@
 $EndComp
 $Comp
-L AGND #PWR029
+L power:AGND #PWR029
 U 1 1 5A25F900
 P 6500 4750
@@
 $EndComp
 $Comp
-L C C33
+L device:C C33
 U 1 1 5A25F914
 P 3950 1900
@@
 $EndComp
 $Comp
-L DGND #PWR030
+L power:DGND #PWR030
 U 1 1 5A25F91B
 P 3700 1700
@@
 $EndComp
 $Comp
-L C C40
+L device:C C40
 U 1 1 5A25F921
 P 7450 5600
@@
 $EndComp
 $Comp
-L C C47
+L device:C C47
 U 1 1 5A25F928
 P 8850 5450
@@
 $EndComp
 $Comp
-L C C48
+L device:C C48
 U 1 1 5A25F92F
 P 8850 6000
@@
 $EndComp
 $Comp
-L AGND #PWR031
+L power:AGND #PWR031
 U 1 1 5A25F936
 P 9100 5700
@@
 $EndComp
 $Comp
-L AGND #PWR032
+L power:AGND #PWR032
 U 1 1 5A25F93C
 P 9100 6250
@@
 $EndComp
 $Comp
-L C C39
+L device:C C39
 U 1 1 5A25F942
 P 7200 5600
@@
 $EndComp
 $Comp
-L CP2 C45
+L device:CP1 C45
 U 1 1 5A25F949
 P 8600 5450
@@
 $EndComp
 $Comp
-L CP2 C46
+L device:CP1 C46
 U 1 1 5A25F950
 P 8600 6000
@@
 $EndComp
 $Comp
-L CP2 C38
+L device:CP1 C38
 U 1 1 5A25F957
 P 6100 4850
@@
 $EndComp
 $Comp
-L CP2 C36
+L device:CP1 C36
 U 1 1 5A25F95E
 P 5950 2450
@@
 $EndComp
 $Comp
-L CP2 C34
+L device:CP1 C34
 U 1 1 5A25F965
 P 4200 1900
@@
 RESET3
 $Comp
-L CP2 C41
+L device:CP1 C41
 U 1 1 5A25F973
 P 7500 3100
@@
 $EndComp
 $Comp
-L CP2 C42
+L device:CP1 C42
 U 1 1 5A25F97A
 P 7500 3850
@@
 $EndComp
 $Comp
-L C C43
+L device:C C43
 U 1 1 5A25F981
 P 7700 3100
@@
 $EndComp
 $Comp
-L C C44
+L device:C C44
 U 1 1 5A25F988
 P 7700 3850
@@
 $EndComp
 $Comp
-L AGND #PWR033
+L power:AGND #PWR033
 U 1 1 5A25F98F
 P 7400 3300
@@
 $EndComp
 $Comp
-L AGND #PWR034
+L power:AGND #PWR034
 U 1 1 5A25F995
 P 7500 4150
@@
 	6000 3350 6550 3350
 Wire Wire Line
-	7150 3450 7800 3450
+	7150 3450 7250 3450
 Wire Wire Line
 	5000 1350 5000 1500
@@
 	5000 5750 5000 5900
 Wire Wire Line
-	7350 5250 7900 5250
-Wire Wire Line
-	7350 5950 7900 5950
+	7350 5250 7700 5250
 Wire Wire Line
 	6550 3550 6000 3550
@@
 Connection ~ 7250 3450
 Wire Wire Line
-	6850 3100 7050 3100
-Wire Wire Line
-	6850 3800 7000 3800
+	6850 3100 6950 3100
+Wire Wire Line
+	6850 3800 6950 3800
 Wire Wire Line
 	7950 3650 7950 3800
 Wire Wire Line
-	5700 2050 5700 2350
+	5700 2050 5700 2200
 Wire Wire Line
 	5400 4700 5400 4850
@@
 	4900 2400 4900 2600
 Wire Wire Line
-	4350 2400 4900 2400
+	4350 2400 4550 2400
 Wire Wire Line
 	4750 2400 4750 2600
@@
 Connection ~ 5700 2300
 Wire Wire Line
-	6150 2200 6150 2450
+	6150 2200 6150 2300
 Wire Wire Line
 	6150 2300 6400 2300
@@
 	5400 4700 5900 4700
 Wire Wire Line
-	5900 4600 5900 4850
-Wire Wire Line
-	6300 4600 6300 4850
+	5900 4600 5900 4700
+Wire Wire Line
+	6300 4600 6300 4700
 Connection ~ 5900 4700
 Wire Wire Line
@@
 Connection ~ 6300 4700
 Wire Wire Line
-	3950 1700 4200 1700
-Wire Wire Line
-	3950 2100 4200 2100
-Wire Wire Line
-	4050 2100 4550 2100
+	3950 1700 4050 1700
 Wire Wire Line
 	4550 2100 4550 2400
 Connection ~ 4550 2400
-Connection ~ 4050 2100
 Wire Wire Line
 	4050 1700 4050 1450
@@
 Connection ~ 4050 1700
 Wire Wire Line
-	8600 5250 8850 5250
+	8600 5250 8700 5250
 Wire Wire Line
 	8600 5650 8850 5650
 Wire Wire Line
-	7850 5800 8850 5800
-Wire Wire Line
 	8600 6200 8850 6200
 Wire Wire Line
-	7200 5400 7450 5400
-Wire Wire Line
-	7200 5800 7450 5800
+	7200 5400 7350 5400
+Wire Wire Line
+	7200 5800 7350 5800
 Wire Wire Line
 	7350 5400 7350 5250
@@
 Wire Wire Line
 	7350 5800 7350 5950
-Connection ~ 7700 5950
 Connection ~ 7350 5800
 Wire Wire Line
-	7700 5950 7850 5950
-Wire Wire Line
 	7850 5950 7850 5800
-Connection ~ 8600 5800
 Wire Wire Line
 	7700 5250 7700 5150
@@
 	8850 5700 9100 5700
 Wire Wire Line
-	8850 5600 8850 5700
+	8850 5600 8850 5650
 Wire Wire Line
 	8850 6250 9100 6250
 Wire Wire Line
-	8850 6150 8850 6250
+	8850 6150 8850 6200
 Wire Wire Line
 	3300 4100 3950 4100
@@
 Connection ~ 7800 5950
 Wire Wire Line
-	7500 2900 7700 2900
-Wire Wire Line
-	7400 3300 7700 3300
-Wire Wire Line
-	7500 3650 7700 3650
-Wire Wire Line
 	7500 4050 7700 4050
-Wire Wire Line
-	7600 2900 6950 2900
 Wire Wire Line
 	6950 2900 6950 3100
 Connection ~ 6950 3100
-Connection ~ 7600 2900
-Wire Wire Line
-	7600 3650 6950 3650
 Wire Wire Line
 	6950 3650 6950 3800
 Connection ~ 6950 3800
-Connection ~ 7600 3650
-Connection ~ 7500 4050
-Connection ~ 7500 3300
-$Comp
-L R R3
+$Comp
+L device:R R3
 U 1 1 5A25FA0F
 P 7250 4550
@@
 $EndComp
 $Comp
-L AGND #PWR035
+L power:AGND #PWR035
 U 1 1 5A25FA16
 P 7000 4650
@@
 $EndComp
 $Comp
-L DGND #PWR036
+L power:DGND #PWR036
 U 1 1 5A25FA1C
 P 7500 4650
@@
 Wire Wire Line
 	8850 5250 8850 5300
+Wire Wire Line
+	7250 3450 7800 3450
+Wire Wire Line
+	4750 2400 4900 2400
+Wire Wire Line
+	5700 2200 5700 2300
+Wire Wire Line
+	5700 2300 5700 2350
+Wire Wire Line
+	6150 2300 6150 2450
+Wire Wire Line
+	5900 4700 5900 4850
+Wire Wire Line
+	6300 4700 6300 4850
+Wire Wire Line
+	4550 2400 4750 2400
+Wire Wire Line
+	4050 1700 4200 1700
+Wire Wire Line
+	7700 5250 7800 5250
+Wire Wire Line
+	7350 5400 7450 5400
+Wire Wire Line
+	7350 5800 7450 5800
+Wire Wire Line
+	8700 5250 8850 5250
+Wire Wire Line
+	7800 5250 7900 5250
+Wire Wire Line
+	6950 3100 7050 3100
+Wire Wire Line
+	6950 3800 7000 3800
+Wire Wire Line
+	8850 6200 8850 6250
+Wire Wire Line
+	8850 5650 8850 5700
+Wire Wire Line
+	7850 5800 8850 5800
+Wire Wire Line
+	7400 3300 7700 3300
+Wire Wire Line
+	3950 2100 4550 2100
+Wire Wire Line
+	7350 5950 7800 5950
+Wire Wire Line
+	7800 5950 7900 5950
+Wire Wire Line
+	6950 2900 7700 2900
+Wire Wire Line
+	6950 3650 7700 3650
 $EndSCHEMATC

Commit message: fixing more borkage
Connections:
- net labels added: +5V
- net labels removed: 3.3V
- wire segments 126 -> 113
Changed lines of the file:
@@
 Text GLabel 5450 4850 2    60   Input ~ 0
 -14V
-Text GLabel 4350 2400 0    60   Input ~ 0
-3.3V
 $Comp
 L power:AGND #PWR026
@@
 L power:DGND #PWR027
 U 1 1 5A25F8E6
-P 4700 4900
-F 0 "#PWR027" H 4700 4900 40  0001 C CNN
-F 1 "DGND" H 4700 4830 40  0000 C CNN
-F 2 "" H 4700 4900 60  0000 C CNN
-F 3 "" H 4700 4900 60  0000 C CNN
-	1    4700 4900
+P 4800 5000
+F 0 "#PWR027" H 4800 5000 40  0001 C CNN
+F 1 "DGND" H 4800 4930 40  0000 C CNN
+F 2 "" H 4800 5000 60  0000 C CNN
+F 3 "" H 4800 5000 60  0000 C CNN
+	1    4800 5000
 	1    0    0    -1
 $EndComp
@@
 	7950 3650 7950 3800
 Wire Wire Line
-	5700 2050 5700 2200
-Wire Wire Line
 	5400 4700 5400 4850
 Wire Wire Line
@@
 	4950 4900 4950 4700
 Wire Wire Line
-	4700 4900 4800 4900
-Wire Wire Line
-	4800 4900 4800 4700
-Wire Wire Line
 	5700 2350 5350 2350
 Wire Wire Line
 	5350 2350 5350 2600
-Wire Wire Line
-	5700 2200 5800 2200
-Connection ~ 5700 2200
 Wire Wire Line
 	5750 2450 5750 2300
@@
 Connection ~ 7350 5800
 Wire Wire Line
-	7850 5950 7850 5800
-Wire Wire Line
 	7700 5250 7700 5150
 Wire Wire Line
@@
 	8850 5700 9100 5700
 Wire Wire Line
-	8850 5600 8850 5650
-Wire Wire Line
 	8850 6250 9100 6250
-Wire Wire Line
-	8850 6150 8850 6200
 Wire Wire Line
 	3300 4100 3950 4100
@@
 	7000 4550 7000 4650
 Wire Wire Line
-	7700 3650 7700 3700
-Wire Wire Line
-	7700 4050 7700 4000
-Wire Wire Line
-	7500 4550 7400 4550
-Wire Wire Line
-	7100 4550 7000 4550
-Wire Wire Line
-	6250 4600 6300 4600
-Wire Wire Line
-	5950 4600 5900 4600
-Wire Wire Line
-	7700 2900 7700 2950
-Wire Wire Line
-	7700 3300 7700 3250
-Wire Wire Line
-	3950 2050 3950 2100
-Wire Wire Line
-	3950 1750 3950 1700
-Wire Wire Line
-	6100 2200 6150 2200
-Wire Wire Line
 	3300 3200 3950 3200
 Wire Wire Line
 	7500 4150 7500 4050
-Wire Wire Line
-	7450 5400 7450 5450
-Wire Wire Line
-	7450 5800 7450 5750
-Wire Wire Line
-	7200 5800 7200 5750
-Wire Wire Line
-	7200 5450 7200 5400
-Wire Wire Line
-	8850 5800 8850 5850
 Connection ~ 8850 6200
 Connection ~ 8850 5650
 Wire Wire Line
-	8850 5250 8850 5300
-Wire Wire Line
 	7250 3450 7800 3450
 Wire Wire Line
 	4750 2400 4900 2400
 Wire Wire Line
+	5700 2300 5700 2350
+Wire Wire Line
+	6150 2300 6150 2450
+Wire Wire Line
+	5900 4700 5900 4850
+Wire Wire Line
+	6300 4700 6300 4850
+Wire Wire Line
+	4550 2400 4750 2400
+Wire Wire Line
+	4050 1700 4200 1700
+Wire Wire Line
+	7700 5250 7800 5250
+Wire Wire Line
+	7350 5400 7450 5400
+Wire Wire Line
+	7350 5800 7450 5800
+Wire Wire Line
+	8700 5250 8850 5250
+Wire Wire Line
+	7800 5250 7900 5250
+Wire Wire Line
+	6950 3100 7050 3100
+Wire Wire Line
+	6950 3800 7000 3800
+Wire Wire Line
+	8850 6200 8850 6250
+Wire Wire Line
+	8850 5650 8850 5700
+Wire Wire Line
+	7850 5800 8600 5800
+Wire Wire Line
+	7400 3300 7500 3300
+Wire Wire Line
+	3950 2100 4200 2100
+Wire Wire Line
+	7350 5950 7800 5950
+Wire Wire Line
+	7800 5950 7850 5950
+Wire Wire Line
+	6950 2900 7500 2900
+Wire Wire Line
+	6950 3650 7500 3650
+Wire Wire Line
+	7850 5800 7850 5950
+Connection ~ 7850 5950
+Wire Wire Line
+	7850 5950 7900 5950
+Connection ~ 8600 5800
+Wire Wire Line
+	8600 5800 8850 5800
+Connection ~ 7500 3650
+Wire Wire Line
+	7500 3650 7700 3650
+Connection ~ 7500 4050
+Connection ~ 7500 2900
+Wire Wire Line
+	7500 2900 7700 2900
+Connection ~ 7500 3300
+Wire Wire Line
+	7500 3300 7700 3300
+Wire Wire Line
+	5700 2050 5700 2200
+Wire Wire Line
+	5750 2200 5700 2200
+Connection ~ 5700 2200
+Wire Wire Line
 	5700 2200 5700 2300
-Wire Wire Line
-	5700 2300 5700 2350
-Wire Wire Line
-	6150 2300 6150 2450
-Wire Wire Line
-	5900 4700 5900 4850
-Wire Wire Line
-	6300 4700 6300 4850
-Wire Wire Line
-	4550 2400 4750 2400
-Wire Wire Line
-	4050 1700 4200 1700
-Wire Wire Line
-	7700 5250 7800 5250
-Wire Wire Line
-	7350 5400 7450 5400
-Wire Wire Line
-	7350 5800 7450 5800
-Wire Wire Line
-	8700 5250 8850 5250
-Wire Wire Line
-	7800 5250 7900 5250
-Wire Wire Line
-	6950 3100 7050 3100
-Wire Wire Line
-	6950 3800 7000 3800
-Wire Wire Line
-	8850 6200 8850 6250
-Wire Wire Line
-	8850 5650 8850 5700
-Wire Wire Line
-	7850 5800 8850 5800
-Wire Wire Line
-	7400 3300 7700 3300
-Wire Wire Line
-	3950 2100 4550 2100
-Wire Wire Line
-	7350 5950 7800 5950
-Wire Wire Line
-	7800 5950 7900 5950
-Wire Wire Line
-	6950 2900 7700 2900
-Wire Wire Line
-	6950 3650 7700 3650
+Connection ~ 4200 2100
+Wire Wire Line
+	4200 2100 4550 2100
+$Comp
+L power:+5V #PWR?
+U 1 1 5A4C4FFF
+P 4350 2350
+F 0 "#PWR?" H 4350 2440 20  0001 C CNN
+F 1 "+5V" H 4346 2478 30  0000 C CNN
+F 2 "" H 4350 2350 60  0001 C CNN
+F 3 "" H 4350 2350 60  0001 C CNN
+	1    4350 2350
+	1    0    0    -1
+$EndComp
+Wire Wire Line
+	4350 2350 4350 2400
+Wire Wire Line
+	4800 4700 4800 5000
 $EndSCHEMATC
