File: stm_pcbs/stm_integrated/IOPW.sch (KiCad schematic (older format))
At the start: 0 parts

Commit message: working on Kicad of 3rd Dec
Parts:
- added P?: CONN_20X2, symbol conn:CONN_20X2
Connections:
- new net +14V: P?.39 (P39)
- new net +5V: P?.31 (P31)
- new net -14V: P?.35 (P35)
- new net ADC_BUSY: P?.15 (P15)
- new net ADC_CONVST: P?.19 (P19)
- new net ADC_RD: P?.17 (P17)
- new net CLR1: P?.4 (P4)
- new net CLR2: P?.12 (P12)
- new net CLR3: P?.20 (P20)
- new net CLR4: P?.9 (P9)
- new net DGND: P?.21 (P21), P?.23 (P23), P?.26 (P26), P?.27 (P27)
- new net LDAC1: P?.6 (P6)
- new net LDAC2: P?.14 (P14)
- new net LDAC3: P?.22 (P22)
- new net LDAC4: P?.11 (P11)
- new net RESET1: P?.2 (P2)
- new net RESET2: P?.10 (P10)
- new net RESET3: P?.18 (P18)
- new net RESET4: P?.7 (P7)
- new net SCLK: P?.1 (P1)
- new net SDIN: P?.3 (P3)
- new net SDO: P?.5 (P5)
- new net SYNC1: P?.8 (P8)
- new net SYNC2: P?.16 (P16)
- new net SYNC3: P?.24 (P24)
- new net SYNC4: P?.13 (P13)
Changed lines of the file:
@@
-EESchema Schematic File Version 2
-LIBS:power
-LIBS:device
-LIBS:transistors
-LIBS:conn
-LIBS:linear
-LIBS:regul
-LIBS:74xx
-LIBS:cmos4000
-LIBS:adc-dac
-LIBS:memory
-LIBS:xilinx
-LIBS:special
-LIBS:microcontrollers
-LIBS:dsp
-LIBS:microchip
-LIBS:analog_switches
-LIBS:motorola
-LIBS:texas
-LIBS:intel
-LIBS:audio
-LIBS:interface
-LIBS:digital-audio
-LIBS:philips
-LIBS:display
-LIBS:cypress
-LIBS:siliconi
-LIBS:opto
-LIBS:atmel
-LIBS:contrib
-LIBS:valves
-LIBS:ad5791
+EESchema Schematic File Version 4
 LIBS:stmshieldfull-cache
-LIBS:powerbrd-cache
-LIBS:LTC1859-cache
-EELAYER 25 0
+EELAYER 26 0
 EELAYER END
 $Descr A4 11693 8268
 encoding utf-8
-Sheet 1 8
+Sheet 8 8
 Title ""
 Date ""
@@
 Comment4 ""
 $EndDescr
+Text GLabel 5950 2800 1    60   Input ~ 0
+ADC_CONVST
+Text GLabel 6050 2800 1    60   Input ~ 0
+ADC_RD
+Text GLabel 6150 2800 1    60   Input ~ 0
+ADC_BUSY
+Text GLabel 6850 2800 1    60   Input ~ 0
+SCLK
+Text GLabel 6750 2800 1    60   Input ~ 0
+SDIN
+Text GLabel 6650 2800 1    60   Input ~ 0
+SDO
+Text GLabel 6550 4900 3    60   Input ~ 0
+SYNC1
+Text GLabel 6650 4900 3    60   Input ~ 0
+LDAC1
+Text GLabel 6750 4900 3    60   Input ~ 0
+CLR1
+Text GLabel 6850 4900 3    60   Input ~ 0
+RESET1
+Wire Wire Line
+	6850 4900 6850 4250
+Wire Wire Line
+	6750 4900 6750 4250
+Wire Wire Line
+	6650 4900 6650 4250
+Wire Wire Line
+	6850 3450 6850 2800
+Wire Wire Line
+	6750 2800 6750 3450
+Wire Wire Line
+	6650 2800 6650 3450
+Wire Wire Line
+	6550 4900 6550 4250
+$Comp
+L conn:CONN_20X2 P?
+U 1 1 5A232155
+P 5900 3850
+F 0 "P?" V 5855 4877 60  0000 L CNN
+F 1 "CONN_20X2" V 5953 4877 50  0000 L CNN
+F 2 "" H 5900 3850 60  0000 C CNN
+F 3 "" H 5900 3850 60  0000 C CNN
+	1    5900 3850
+	0    1    1    0
+$EndComp
+Text GLabel 6150 4900 3    60   Input ~ 0
+SYNC2
+Text GLabel 6250 4900 3    60   Input ~ 0
+LDAC2
+Text GLabel 6350 4900 3    60   Input ~ 0
+CLR2
+Text GLabel 6450 4900 3    60   Input ~ 0
+RESET2
+Wire Wire Line
+	6450 4900 6450 4250
+Wire Wire Line
+	6350 4900 6350 4250
+Wire Wire Line
+	6250 4900 6250 4250
+Wire Wire Line
+	6150 4900 6150 4250
+Text GLabel 5750 4900 3    60   Input ~ 0
+SYNC3
+Text GLabel 5850 4900 3    60   Input ~ 0
+LDAC3
+Text GLabel 5950 4900 3    60   Input ~ 0
+CLR3
+Text GLabel 6050 4900 3    60   Input ~ 0
+RESET3
+Wire Wire Line
+	6050 4900 6050 4250
+Wire Wire Line
+	5950 4900 5950 4250
+Wire Wire Line
+	5850 4900 5850 4250
+Wire Wire Line
+	5750 4900 5750 4250
+Text GLabel 6250 2800 1    60   Input ~ 0
+SYNC4
+Text GLabel 6350 2800 1    60   Input ~ 0
+LDAC4
+Text GLabel 6450 2800 1    60   Input ~ 0
+CLR4
+Text GLabel 6550 2800 1    60   Input ~ 0
+RESET4
+Wire Wire Line
+	6550 2800 6550 3450
+Wire Wire Line
+	6450 2800 6450 3450
+Wire Wire Line
+	6350 2800 6350 3450
+Wire Wire Line
+	6250 2800 6250 3450
+Wire Wire Line
+	6150 2800 6150 3450
+Wire Wire Line
+	6050 2800 6050 3450
+Wire Wire Line
+	5950 2800 5950 3450
+$Comp
+L +5V #PWR?
+U 1 1 5A2349B8
+P 5350 4350
+AR Path="/5A2349B8" Ref="#PWR?"  Part="1"
+AR Path="/5A25A549/5A2349B8" Ref="#PWR?"  Part="1"
+F 0 "#PWR?" H 5350 4440 20  0001 C CNN
+F 1 "+5V" H 5347 4477 30  0000 C CNN
+F 2 "" H 5350 4350 60  0001 C CNN
+F 3 "" H 5350 4350 60  0001 C CNN
+	1    5350 4350
+	-1   0    0    1
+$EndComp
+Text GLabel 4950 4350 3    60   Input ~ 0
++14V
+Text GLabel 5150 4350 3    60   Input ~ 0
+-14V
+$Comp
+L DGND #PWR?
+U 1 1 5A2352DB
+P 7450 5000
+AR Path="/5A2352DB" Ref="#PWR?"  Part="1"
+AR Path="/5A25A549/5A2352DB" Ref="#PWR?"  Part="1"
+F 0 "#PWR?" H 7450 5000 40  0001 C CNN
+F 1 "DGND" H 7450 5067 40  0000 C CNN
+F 2 "" H 7450 5000 60  0001 C CNN
+F 3 "" H 7450 5000 60  0001 C CNN
+	1    7450 5000
+	1    0    0    -1
+$EndComp
+$Comp
+L GND #PWR?
+U 1 1 5A23531C
+P 5550 4400
+AR Path="/5A23531C" Ref="#PWR?"  Part="1"
+AR Path="/5A25A549/5A23531C" Ref="#PWR?"  Part="1"
+F 0 "#PWR?" H 5550 4400 30  0001 C CNN
+F 1 "GND" H 5550 4330 30  0001 C CNN
+F 2 "" H 5550 4400 60  0001 C CNN
+F 3 "" H 5550 4400 60  0001 C CNN
+	1    5550 4400
+	1    0    0    -1
+$EndComp
+$Comp
+L GND #PWR?
+U 1 1 5A235335
+P 7700 5000
+AR Path="/5A235335" Ref="#PWR?"  Part="1"
+AR Path="/5A25A549/5A235335" Ref="#PWR?"  Part="1"
+F 0 "#PWR?" H 7700 5000 30  0001 C CNN
+F 1 "GND" H 7700 4930 30  0001 C CNN
+F 2 "" H 7700 5000 60  0001 C CNN
+F 3 "" H 7700 5000 60  0001 C CNN
+	1    7700 5000
+	1    0    0    -1
+$EndComp
+Wire Wire Line
+	7700 5000 7700 4900
+Wire Wire Line
+	7700 4900 7450 4900
+Wire Wire Line
+	7450 4900 7450 5000
+$Comp
+L DGND #PWR?
+U 1 1 5A2355CE
+P 5700 3150
+AR Path="/5A2355CE" Ref="#PWR?"  Part="1"
+AR Path="/5A25A549/5A2355CE" Ref="#PWR?"  Part="1"
+F 0 "#PWR?" H 5700 3150 40  0001 C CNN
+F 1 "DGND" H 5700 3217 40  0000 C CNN
+F 2 "" H 5700 3150 60  0001 C CNN
+F 3 "" H 5700 3150 60  0001 C CNN
+	1    5700 3150
+	1    0    0    -1
+$EndComp
+Wire Wire Line
+	5700 3150 5700 3100
+Wire Wire Line
+	5700 3100 5850 3100
+Wire Wire Line
+	5850 3100 5850 3450
+Wire Wire Line
+	5850 3450 5750 3450
+Wire Wire Line
+	5650 4250 5650 3850
+Wire Wire Line
+	5650 3850 5750 3850
+Wire Wire Line
+	5750 3850 5750 3450
+Wire Wire Line
+	5150 3450 5150 4350
+Wire Wire Line
+	4950 3450 4950 4350
+Wire Wire Line
+	5350 3450 5350 4350
+Wire Wire Line
+	5550 3450 5550 4400
 $EndSCHEMATC

Commit message: fixing more borkage
Parts:
- P6: renamed from P?; footprint (none) -> Connectors_IDC:IDC-Header_2x20_Pitch2.54mm_Straight
Changed lines of the file:
@@
 	6550 4900 6550 4250
 $Comp
-L conn:CONN_20X2 P?
+L conn:CONN_20X2 P6
 U 1 1 5A232155
 P 5900 3850
-F 0 "P?" V 5855 4877 60  0000 L CNN
+F 0 "P6" V 5855 4877 60  0000 L CNN
 F 1 "CONN_20X2" V 5953 4877 50  0000 L CNN
-F 2 "" H 5900 3850 60  0000 C CNN
+F 2 "Connectors_IDC:IDC-Header_2x20_Pitch2.54mm_Straight" H 5900 3850 60  0001 C CNN
 F 3 "" H 5900 3850 60  0000 C CNN
 	1    5900 3850
@@
 P 5350 4350
 AR Path="/5A2349B8" Ref="#PWR?"  Part="1"
-AR Path="/5A25A549/5A2349B8" Ref="#PWR?"  Part="1"
-F 0 "#PWR?" H 5350 4440 20  0001 C CNN
+AR Path="/5A25A549/5A2349B8" Ref="#PWR074"  Part="1"
+F 0 "#PWR074" H 5350 4440 20  0001 C CNN
 F 1 "+5V" H 5347 4477 30  0000 C CNN
 F 2 "" H 5350 4350 60  0001 C CNN
@@
 P 7450 5000
 AR Path="/5A2352DB" Ref="#PWR?"  Part="1"
-AR Path="/5A25A549/5A2352DB" Ref="#PWR?"  Part="1"
-F 0 "#PWR?" H 7450 5000 40  0001 C CNN
+AR Path="/5A25A549/5A2352DB" Ref="#PWR075"  Part="1"
+F 0 "#PWR075" H 7450 5000 40  0001 C CNN
 F 1 "DGND" H 7450 5067 40  0000 C CNN
 F 2 "" H 7450 5000 60  0001 C CNN
@@
 P 5550 4400
 AR Path="/5A23531C" Ref="#PWR?"  Part="1"
-AR Path="/5A25A549/5A23531C" Ref="#PWR?"  Part="1"
-F 0 "#PWR?" H 5550 4400 30  0001 C CNN
+AR Path="/5A25A549/5A23531C" Ref="#PWR076"  Part="1"
+F 0 "#PWR076" H 5550 4400 30  0001 C CNN
 F 1 "GND" H 5550 4330 30  0001 C CNN
 F 2 "" H 5550 4400 60  0001 C CNN
@@
 P 7700 5000
 AR Path="/5A235335" Ref="#PWR?"  Part="1"
-AR Path="/5A25A549/5A235335" Ref="#PWR?"  Part="1"
-F 0 "#PWR?" H 7700 5000 30  0001 C CNN
+AR Path="/5A25A549/5A235335" Ref="#PWR077"  Part="1"
+F 0 "#PWR077" H 7700 5000 30  0001 C CNN
 F 1 "GND" H 7700 4930 30  0001 C CNN
 F 2 "" H 7700 5000 60  0001 C CNN
@@
 P 5700 3150
 AR Path="/5A2355CE" Ref="#PWR?"  Part="1"
-AR Path="/5A25A549/5A2355CE" Ref="#PWR?"  Part="1"
-F 0 "#PWR?" H 5700 3150 40  0001 C CNN
+AR Path="/5A25A549/5A2355CE" Ref="#PWR078"  Part="1"
+F 0 "#PWR078" H 5700 3150 40  0001 C CNN
 F 1 "DGND" H 5700 3217 40  0000 C CNN
 F 2 "" H 5700 3150 60  0001 C CNN

Commit message: tidying up boards, adding all DAC signals.
Changed lines of the file:
@@
 $EndComp
 $Comp
-L GND #PWR?
+L power:GND #PWR?
 U 1 1 5A23531C
 P 5550 4400
@@
 $EndComp
 $Comp
-L GND #PWR?
+L power:GND #PWR?
 U 1 1 5A235335
 P 7700 5000

Commit message: Using LTZ1000 (A9 board)
Parts:
- added R11: 0, Resistors_SMD:R_0201_NoSilk, symbol device:R
Connections:
- net +14V: now also P6.40 (P40)
- net +5V: now also P6.32 (P32)
- net -14V: now also P6.36 (P36)
- net DGND: now also R11.2; no longer P6.27 (P27)
- net GND: now reaches P6.28 (P28)
- net GND: now also P6.27 (P27), R11.1
Changed lines of the file:
@@
 	5950 2800 5950 3450
 $Comp
-L +5V #PWR?
+L stmshieldfull-rescue:+5V-RESCUE-stmshieldfull #PWR?
 U 1 1 5A2349B8
 P 5350 4350
@@
 -14V
 $Comp
-L DGND #PWR?
+L stmshieldfull-rescue:DGND-RESCUE-stmshieldfull #PWR?
 U 1 1 5A2352DB
-P 7450 5000
+P 7300 4750
 AR Path="/5A2352DB" Ref="#PWR?"  Part="1"
 AR Path="/5A25A549/5A2352DB" Ref="#PWR075"  Part="1"
-F 0 "#PWR075" H 7450 5000 40  0001 C CNN
-F 1 "DGND" H 7450 5067 40  0000 C CNN
-F 2 "" H 7450 5000 60  0001 C CNN
-F 3 "" H 7450 5000 60  0001 C CNN
-	1    7450 5000
+F 0 "#PWR075" H 7300 4750 40  0001 C CNN
+F 1 "DGND" H 7300 4817 40  0000 C CNN
+F 2 "" H 7300 4750 60  0001 C CNN
+F 3 "" H 7300 4750 60  0001 C CNN
+	1    7300 4750
 	1    0    0    -1
 $EndComp
@@
 L power:GND #PWR?
 U 1 1 5A235335
-P 7700 5000
+P 7800 4750
 AR Path="/5A235335" Ref="#PWR?"  Part="1"
 AR Path="/5A25A549/5A235335" Ref="#PWR077"  Part="1"
-F 0 "#PWR077" H 7700 5000 30  0001 C CNN
-F 1 "GND" H 7700 4930 30  0001 C CNN
-F 2 "" H 7700 5000 60  0001 C CNN
-F 3 "" H 7700 5000 60  0001 C CNN
-	1    7700 5000
+F 0 "#PWR077" H 7800 4750 30  0001 C CNN
+F 1 "GND" H 7800 4680 30  0001 C CNN
+F 2 "" H 7800 4750 60  0001 C CNN
+F 3 "" H 7800 4750 60  0001 C CNN
+	1    7800 4750
 	1    0    0    -1
 $EndComp
 Wire Wire Line
-	7700 5000 7700 4900
+	7800 4750 7800 4650
 Wire Wire Line
-	7700 4900 7450 4900
-Wire Wire Line
-	7450 4900 7450 5000
+	7300 4650 7300 4750
 $Comp
-L DGND #PWR?
+L stmshieldfull-rescue:DGND-RESCUE-stmshieldfull #PWR?
 U 1 1 5A2355CE
 P 5700 3150
@@
 Wire Wire Line
 	5750 3850 5750 3450
+$Comp
+L device:R R11
+U 1 1 5A5F8F90
+P 7550 4650
+F 0 "R11" V 7365 4650 40  0000 C CNN
+F 1 "0" V 7441 4650 40  0000 C CNN
+F 2 "Resistors_SMD:R_0201_NoSilk" V 7480 4650 30  0001 C CNN
+F 3 "" H 7550 4650 30  0000 C CNN
+	1    7550 4650
+	0    1    1    0
+$EndComp
 Wire Wire Line
-	5150 3450 5150 4350
+	5150 3450 5150 4250
+Connection ~ 5150 4250
 Wire Wire Line
-	4950 3450 4950 4350
+	5150 4250 5150 4350
 Wire Wire Line
-	5350 3450 5350 4350
+	4950 3450 4950 4250
+Connection ~ 4950 4250
 Wire Wire Line
-	5550 3450 5550 4400
+	4950 4250 4950 4350
+Wire Wire Line
+	5350 3450 5350 4250
+Connection ~ 5350 4250
+Wire Wire Line
+	5350 4250 5350 4350
+Wire Wire Line
+	5550 3450 5550 4250
+Connection ~ 5550 4250
+Wire Wire Line
+	5550 4250 5550 4400
 $EndSCHEMATC

Commit message: fixed issue with DAC (opamp wiring was wrong)
Parts:
- added R12: 0, Resistors_SMD:R_0201_NoSilk, symbol device:R
Connections:
- net GND: now also R12.1
- new net AGND: R12.2
Changed lines of the file:
@@
 Wire Wire Line
 	5550 4250 5550 4400
+$Comp
+L LTC1859:AGND #PWR059
+U 1 1 5A2A6948
+P 7300 5150
+F 0 "#PWR059" H 7300 5150 40  0001 C CNN
+F 1 "AGND" H 7295 5225 50  0000 C CNN
+F 2 "" H 7300 5150 60  0000 C CNN
+F 3 "" H 7300 5150 60  0000 C CNN
+	1    7300 5150
+	1    0    0    -1
+$EndComp
+$Comp
+L device:R R12
+U 1 1 5A2A696B
+P 7550 5050
+F 0 "R12" V 7365 5050 40  0000 C CNN
+F 1 "0" V 7441 5050 40  0000 C CNN
+F 2 "Resistors_SMD:R_0201_NoSilk" V 7480 5050 30  0001 C CNN
+F 3 "" H 7550 5050 30  0000 C CNN
+	1    7550 5050
+	0    1    1    0
+$EndComp
+$Comp
+L power:GND #PWR083
+U 1 1 5A2A69AB
+P 7800 5150
+F 0 "#PWR083" H 7800 5150 30  0001 C CNN
+F 1 "GND" H 7800 5080 30  0001 C CNN
+F 2 "" H 7800 5150 60  0001 C CNN
+F 3 "" H 7800 5150 60  0001 C CNN
+	1    7800 5150
+	1    0    0    -1
+$EndComp
+Wire Wire Line
+	7800 5150 7800 5050
+Wire Wire Line
+	7300 5150 7300 5050
 $EndSCHEMATC
